File: UNO/eagle-design/vOne - UNO/vONE-UNO.brd (EAGLE design)
At the start: 119.4 x 53.3 mm, 24 parts, among them IC1 ATMEGA328-20P, IC2 7805T, IC4 LM1117MP-3.3, Q1 16 MHz

Commit message: Final design complete
Parts:
- added C5: 100 NF, capacitor-wima:C2.5-3
- added JP2: (no value), adafruit:1X06-BIG
Connections:
- new net N$21: C5.2, JP2.6
- net 0: now also JP2.1
- net N$10: now also JP2.4
- net N$2: now also C5.1
- net N$32: now also JP2.3
- net N$37: now also JP2.5
Routing:
- net N$37: track 50.0 -> 117.9 mm
- net N$10: track 42.8 -> 108.2 mm
- net N$32: track 116.2 -> 152.8 mm, vias 0 -> 1
- net 0: track 185.0 -> 221.4 mm
- net N$21: track 0.00 -> 8.67 mm
- net N$2: track 60.7 -> 66.8 mm
- net N$5: track 55.0 -> 56.1 mm
- net N$28: track 84.2 -> 85.0 mm
Other:
- board text added: "100 NF"
- board text added: "16 Mhz"
- board text added: "22 pF"
- board text added: "A0"
- board text added: "A1"
- board text added: "A2"
- board text added: "A3"
- board text added: "A4"
- board text added: "A5"
- board text added: "ATMEGA328P"
- board text added: "CTS"
- board text added: "D0"
- board text added: "D1"
- board text added: "D10"
- board text added: "D11"
- board text added: "D12"
- board text added: "D13"
- board text added: "D2"
- board text added: "D3"
- board text added: "D4"
- board text added: "D5"
- board text added: "D6"
- board text added: "D7"
- board text added: "D8"
- board text added: "D9"
- board text added: "DTR"
- board text added: "GND"
- board text added: "VCC"
