File: vone-uno/vONE-UNO.brd (EAGLE design)
At the start: 119.4 x 53.3 mm, 27 parts, among them IC1 ATMEGA328-20P, IC2 7805T, IC4 LM1117MP-3.3, Q1 16 MHz

Commit message: Fixed design error
Parts:
- moved C6 85.2 mm to (83.8, 69.5), turned to 90 degrees
Routing:
- net N$27: track 0.00 -> 19.0 mm
- net N$3: track 24.4 -> 35.0 mm
- net N$32: track 149.0 -> 151.3 mm
Other:
- board text added: "sashwat.in"
- board text removed: "sashwat.in | sashuu6.github.io"
Changed lines of the file:
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@@
 <drawing>
 <settings>
-<setting alwaysvectorfont="no"/>
+<setting alwaysvectorfont="yes"/>
 <setting verticaltext="up"/>
 </settings>
@@
 <layer number="27" name="tValues" color="7" fill="1" visible="yes" active="yes"/>
 <layer number="28" name="bValues" color="7" fill="1" visible="yes" active="yes"/>
-<layer number="29" name="tStop" color="7" fill="3" visible="no" active="yes"/>
-<layer number="30" name="bStop" color="7" fill="6" visible="no" active="yes"/>
+<layer number="29" name="tStop" color="7" fill="3" visible="yes" active="yes"/>
+<layer number="30" name="bStop" color="7" fill="6" visible="yes" active="yes"/>
 <layer number="31" name="tCream" color="7" fill="4" visible="no" active="yes"/>
 <layer number="32" name="bCream" color="7" fill="5" visible="no" active="yes"/>
@@
 <text x="5.08" y="57.15" size="2.54" layer="21">vONE
 Ver 2.0</text>
-<text x="116.84" y="57.15" size="1.778" layer="21" rot="R90">sashwat.in | sashuu6.github.io</text>
+<text x="116.713" y="68.199" size="1.778" layer="21" rot="R90">sashwat.in</text>
 <text x="1.27" y="92.71" size="1.778" layer="21">9V AC/DC</text>
 <text x="6.35" y="74.93" size="0.8128" layer="21">1N4007</text>
@@
 <text x="90.297" y="65.532" size="0.635" layer="25">22 pF</text>
 <text x="30.353" y="53.213" size="0.635" layer="25">100 NF</text>
+<polygon width="0.1524" layer="29">
+<vertex x="20.32" y="98.425"/>
+<vertex x="30.607" y="98.425"/>
+<vertex x="30.607" y="96.52"/>
+<vertex x="29.718" y="96.52"/>
+<vertex x="29.718" y="94.996"/>
+<vertex x="30.607" y="94.996"/>
+<vertex x="30.607" y="91.694"/>
+<vertex x="20.193" y="91.694"/>
+<vertex x="20.193" y="94.996"/>
+<vertex x="21.082" y="94.996"/>
+<vertex x="21.082" y="96.52"/>
+<vertex x="20.193" y="96.52"/>
+<vertex x="20.193" y="98.425"/>
+</polygon>
+<polygon width="0.1524" layer="30">
+<vertex x="20.193" y="98.425"/>
+<vertex x="30.607" y="98.425"/>
+<vertex x="30.607" y="96.52"/>
+<vertex x="29.718" y="96.52"/>
+<vertex x="29.718" y="94.996"/>
+<vertex x="30.607" y="94.996"/>
+<vertex x="30.607" y="91.694"/>
+<vertex x="20.193" y="91.694"/>
+<vertex x="20.193" y="94.996"/>
+<vertex x="21.082" y="94.996"/>
+<vertex x="21.082" y="96.52"/>
+<vertex x="20.193" y="96.52"/>
+</polygon>
 </plain>
 <attributes>
@@
 <attribute name="VALUE" x="34.671" y="58.928" size="1.27" layer="27" ratio="10" rot="R180"/>
 </element>
-<element name="C6" library="capacitor-wima" library_urn="urn:adsk.eagle:library:116" package="C2.5-3" package3d_urn="urn:adsk.eagle:package:5436/1" value="100nF" x="2.413" y="44.45" smashed="yes">
-<attribute name="NAME" x="0.762" y="46.228" size="1.27" layer="25" ratio="10"/>
-<attribute name="POPULARITY" value="38" x="2.413" y="44.45" size="1.778" layer="27" display="off"/>
-<attribute name="VALUE" x="0.762" y="41.402" size="1.27" layer="27" ratio="10"/>
+<element name="C6" library="capacitor-wima" library_urn="urn:adsk.eagle:library:116" package="C2.5-3" package3d_urn="urn:adsk.eagle:package:5436/1" value="100nF" x="83.82" y="69.469" smashed="yes" rot="R90">
+<attribute name="NAME" x="82.042" y="67.818" size="1.27" layer="25" ratio="10" rot="R90"/>
+<attribute name="POPULARITY" value="38" x="83.82" y="69.469" size="1.778" layer="27" rot="R90" display="off"/>
+<attribute name="VALUE" x="86.868" y="67.818" size="1.27" layer="27" ratio="10" rot="R90"/>
 </element>
 </elements>
@@
 <wire x1="91.44" y1="62.23" x2="90.17" y2="63.5" width="0.1524" layer="1"/>
 <contactref element="C6" pad="1"/>
-<wire x1="1.143" y1="44.45" x2="90.17" y2="63.5" width="0" layer="19" extent="1-1"/>
+<wire x1="83.82" y1="68.199" x2="83.82" y2="64.262" width="0.1524" layer="16"/>
+<wire x1="83.82" y1="64.262" x2="84.582" y2="63.5" width="0.1524" layer="16"/>
+<wire x1="84.582" y1="63.5" x2="90.17" y2="63.5" width="0.1524" layer="16"/>
 </signal>
 <signal name="N$2">
@@
 <wire x1="68.58" y1="93.98" x2="66.04" y2="93.98" width="0.1524" layer="1"/>
 <wire x1="66.04" y1="93.98" x2="63.5" y2="93.98" width="0.1524" layer="1"/>
-<wire x1="88.9" y1="86.36" x2="87.63" y2="85.09" width="0.1524" layer="1"/>
-<wire x1="87.63" y1="81.28" x2="86.36" y2="80.01" width="0.1524" layer="1"/>
-<wire x1="87.63" y1="85.09" x2="87.63" y2="81.28" width="0.1524" layer="1"/>
 <wire x1="27.94" y1="80.01" x2="33.02" y2="74.93" width="0.3556" layer="1"/>
 <wire x1="33.02" y1="74.93" x2="54.61" y2="74.93" width="0.3556" layer="1"/>
@@
 <wire x1="33.02" y1="63.5" x2="33.02" y2="72.39" width="0.3556" layer="16"/>
 <wire x1="33.02" y1="74.93" x2="33.02" y2="72.39" width="0.3556" layer="1"/>
-<wire x1="88.9" y1="86.36" x2="91.44" y2="87.63" width="0" layer="19" extent="1-1"/>
+<wire x1="86.36" y1="80.01" x2="86.36" y2="81.026" width="0.1524" layer="1"/>
+<wire x1="86.36" y1="81.026" x2="91.44" y2="86.106" width="0.1524" layer="1"/>
+<wire x1="91.44" y1="86.106" x2="91.44" y2="87.63" width="0.1524" layer="1"/>
 </signal>
 <signal name="N$21">
@@
 <contactref element="IC1" pad="21"/>
 <contactref element="C6" pad="2"/>
-<wire x1="3.683" y1="44.45" x2="88.9" y2="87.63" width="0" layer="19" extent="1-1"/>
+<wire x1="88.9" y1="87.63" x2="88.9" y2="85.598" width="0.1524" layer="16"/>
+<wire x1="83.82" y1="74.295" x2="83.82" y2="70.739" width="0.1524" layer="16"/>
+<wire x1="88.9" y1="85.598" x2="87.376" y2="84.074" width="0.1524" layer="16"/>
+<wire x1="87.376" y1="84.074" x2="87.376" y2="77.851" width="0.1524" layer="16"/>
+<wire x1="87.376" y1="77.851" x2="83.82" y2="74.295" width="0.1524" layer="16"/>
+</signal>
+<signal name="N$33">
+<via x="20.955" y="97.536" extent="1-16" drill="0.35"/>
+</signal>
+<signal name="N$35">
+<via x="22.225" y="97.536" extent="1-16" drill="0.35"/>
+</signal>
+<signal name="N$38">
+<via x="22.225" y="96.266" extent="1-16" drill="0.35"/>
+</signal>
+<signal name="N$39">
+<via x="22.225" y="95.123" extent="1-16" drill="0.35"/>
+</signal>
+<signal name="N$40">
+<via x="22.225" y="93.98" extent="1-16" drill="0.35"/>
+</signal>
+<signal name="N$41">
+<via x="20.955" y="93.98" extent="1-16" drill="0.35"/>
+</signal>
+<signal name="N$42">
+<via x="20.955" y="92.837" extent="1-16" drill="0.35"/>
+</signal>
+<signal name="N$43">
+<via x="22.225" y="92.837" extent="1-16" drill="0.35"/>
+</signal>
+<signal name="N$44">
+<via x="23.368" y="97.536" extent="1-16" drill="0.35"/>
+</signal>
+<signal name="N$45">
+<via x="27.432" y="97.536" extent="1-16" drill="0.35"/>
+</signal>
+<signal name="N$46">
+<via x="28.575" y="97.536" extent="1-16" drill="0.35"/>
+</signal>
+<signal name="N$47">
+<via x="29.718" y="97.536" extent="1-16" drill="0.35"/>
+</signal>
+<signal name="N$48">
+<via x="28.702" y="96.266" extent="1-16" drill="0.35"/>
+</signal>
+<signal name="N$49">
+<via x="28.829" y="94.996" extent="1-16" drill="0.35"/>
+</signal>
+<signal name="N$50">
+<via x="28.829" y="93.853" extent="1-16" drill="0.35"/>
+</signal>
+<signal name="N$51">
+<via x="29.972" y="93.853" extent="1-16" drill="0.35"/>
+</signal>
+<signal name="N$52">
+<via x="29.972" y="92.583" extent="1-16" drill="0.35"/>
+</signal>
+<signal name="N$53">
+<via x="28.829" y="92.583" extent="1-16" drill="0.35"/>
+</signal>
+<signal name="N$54">
+<via x="27.686" y="92.583" extent="1-16" drill="0.35"/>
+</signal>
+<signal name="N$55">
+<via x="23.495" y="92.329" extent="1-16" drill="0.35"/>
 </signal>
 </signals>

Commit message: Updated design
Routing:
- net N$5: track 56.1 -> 58.9 mm
- net N$6: track 47.4 -> 49.5 mm
- net N$23: track 38.6 -> 39.9 mm
- net N$3: track 35.0 -> 36.4 mm
- net N$22: track 33.6 -> 34.4 mm
- net N$4: track 57.2 -> 56.7 mm
- net N$37: track 117.9 -> 118.5 mm
Other:
- board text added: "100nF"
- board text added: "3.3V"
- board text added: "5V"
